File: kiCAD/kiCAD.kicad_sch (KiCad schematic)
At the start: 11 parts, among them J1 Analog, J2 Digital, Q1 2N2222

Commit message: Minor update
Updated transitor name with BC547
Parts:
- Q1: value 2N2222 -> 2N2222 - BC547
Changed lines of the file:
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@@
 			)
 		)
-		(property "Value" "2N2222"
+		(property "Value" "2N2222 - BC547"
 			(at 93.98 36.83 90)
 			(effects

Commit message: Updated models
Updated models to figure out last improvements.
Parts:
- MPU-6050, Nidec_24H404H160: value ~ -> (none)
